Commit message: added current calibraded pr2 urdf and renamed odom to odom_combined in urdf with odom joints

File: iai_pr2_description/robots/pr2_with_odom_joints.xacro (robot description, xacro)
@@ -1,8 +1,8 @@
 <?xml version="1.0" ?>
 <robot xmlns:xacro="http://www.ros.org/wiki/xacro" name="pr2">
-  <xacro:include filename="$(find iai_pr2_description)/robots/pr2_calibrated_with_ft.xml"/>
-  <link name="odom"/>
+  <xacro:include filename="$(find iai_pr2_description)/robots/pr2_calibrated_with_ft2.xml"/>
+  <link name="odom_combined"/>
   <joint name="odom_x_joint" type="prismatic">
-    <parent link="odom"/>
+    <parent link="odom_combined"/>
     <child link="odom_x_frame"/>
     <axis xyz="1 0 0"/>

Commit message: added catkin-melodic.rosinstall

File: iai_pr2_description/robots/pr2_with_odom_joints.xacro (robot description, xacro)
@@ -11,5 +11,5 @@
           velocity: slow walking speed is 3-4km/hour ~= 1m/s
           effort: reach max speed within 1s, Boxy has a mass of 200kg, so Fmax=200kg*1m/s2 -->
-    <limit effort="200" lower="-1000" upper="1000" velocity="0.1"/>
+    <limit effort="200" lower="-1000" upper="1000" velocity="1"/>
   </joint>
   <link name="odom_x_frame"/>
@@ -22,5 +22,5 @@
            velocity: slow walking speed is 3-4km/hour ~= 1m/s
            effort: reach max speed within 1s, Boxy has a mass of 200kg, so Fmax=200kg*1m/s2 -->
-    <limit effort="200" lower="-1000" upper="1000" velocity="0.1"/>
+    <limit effort="200" lower="-1000" upper="1000" velocity="1"/>
   </joint>
   <link name="odom_y_frame"/>
@@ -32,5 +32,5 @@
            velocity: one slow complete turn around in 5-6s, so 6.2rad/6s ~= 1rad/s
            effort: reach max speed within 1s, Boxy has a mass of 200kg and a diagonale of 1m, so Fmax=200kg*1m*1m/s2 -->
-    <limit effort="200" velocity="0.2"/>
+    <limit effort="200" velocity="1"/>
   </joint>
 </robot>

Commit message: set pr2s translational velocity limits to 0.5 in the urdf

File: iai_pr2_description/robots/pr2_with_odom_joints.xacro (robot description, xacro)
@@ -11,5 +11,5 @@
           velocity: slow walking speed is 3-4km/hour ~= 1m/s
           effort: reach max speed within 1s, Boxy has a mass of 200kg, so Fmax=200kg*1m/s2 -->
-    <limit effort="200" lower="-1000" upper="1000" velocity="1"/>
+    <limit effort="200" lower="-1000" upper="1000" velocity="0.5"/>
   </joint>
   <link name="odom_x_frame"/>
@@ -22,5 +22,5 @@
            velocity: slow walking speed is 3-4km/hour ~= 1m/s
            effort: reach max speed within 1s, Boxy has a mass of 200kg, so Fmax=200kg*1m/s2 -->
-    <limit effort="200" lower="-1000" upper="1000" velocity="1"/>
+    <limit effort="200" lower="-1000" upper="1000" velocity="0.5"/>
   </joint>
   <link name="odom_y_frame"/>
@@ -32,5 +32,5 @@
            velocity: one slow complete turn around in 5-6s, so 6.2rad/6s ~= 1rad/s
            effort: reach max speed within 1s, Boxy has a mass of 200kg and a diagonale of 1m, so Fmax=200kg*1m*1m/s2 -->
-    <limit effort="200" velocity="1"/>
+    <limit effort="200" velocity="0.2"/>
   </joint>
 </robot>

Commit message: [description] increased odom rotational max vel to 0.4rad/s

File: iai_pr2_description/robots/pr2_with_odom_joints.xacro (robot description, xacro)
@@ -32,5 +32,5 @@
            velocity: one slow complete turn around in 5-6s, so 6.2rad/6s ~= 1rad/s
            effort: reach max speed within 1s, Boxy has a mass of 200kg and a diagonale of 1m, so Fmax=200kg*1m*1m/s2 -->
-    <limit effort="200" velocity="0.2"/>
+    <limit effort="200" velocity="0.4"/>
   </joint>
 </robot>
