Commit message: added real time controllers to mujoco config

File: iai_pr2_description/robots/pr2.urdf (robot description, URDF)
Before this commit: robot pr2, 95 links, 94 joints
Links:
- added link head_mount_kinect2_ir_optical_frame
- added link head_mount_kinect2_rgb_optical_frame
- link l_force_torque_link: geometry collision cylinder length=0.0356 radius=0.0225; visual cylinder length=0.0356 radius=0.0225
Joints:
- added joint head_mount_kinect2_ir_optical_frame_joint: type fixed, parent head_mount_kinect2_rgb_optical_frame, child head_mount_kinect2_ir_optical_frame, origin xyz=-0.050972994874597992 0.00017844406311044261 0.0013319122998533958 rpy=0.0023123703682906313 0.0056320953034389425 0.0022080453816523005
- added joint head_mount_kinect2_rgb_optical_frame_joint: type fixed, parent high_def_optical_frame, child head_mount_kinect2_rgb_optical_frame, origin xyz=-0.017815 -0.064648 -0.037164 rpy=6.262691 0.000163 0.005596
- joint head_mount_kinect_rgb_joint: origin xyz=-0.016464580011 -0.024840302033 -0.015501555887 rpy=-0.009197234917 -0.03162989289 -0.000024986557 -> xyz=-0.011274983694 -0.024595566211 -0.010102622757 rpy=-0.006362360178 -0.036288968859 -0.003498282839
- joint high_def_frame_joint: origin xyz=0.037305871189 -0.109084466748 0.051107786118 rpy=-0.013344088743 -0.002157650878 0.00598407071 -> xyz=0.044490865137 -0.110991674247 0.05733962096 rpy=-0.010992974243 -0.007224184883 0.00316695458
- joint l_forearm_cam_frame_joint: origin xyz=0.143534195191 0.005377510982 0.038210342235 rpy=-1.538533018262 -0.563330072035 -0.015596777949 -> xyz=0.144227112237 -0.007018878517 0.035421631733 rpy=-1.570660881614 -0.556339414268 0.008700049687
- joint l_gripper_l_finger_tip_joint: mimic (none) -> joint=l_gripper_l_finger_joint multiplier=1 offset=0
- joint l_gripper_r_finger_joint: mimic (none) -> joint=l_gripper_l_finger_joint multiplier=1 offset=0
- joint l_gripper_r_finger_tip_joint: mimic (none) -> joint=l_gripper_l_finger_joint multiplier=1 offset=0
- joint laser_tilt_joint: origin xyz=0 0 0.028389479248 rpy=0 0 -0.007935244203 -> xyz=0 0 0.02920161101 rpy=0 0 -0.011866389294
- joint narrow_stereo_frame_joint: origin xyz=0.036004211982 0.059339423616 0.046128460576 rpy=-0.006360148572 -0.007022640169 0.00538386839 -> xyz=0.043113072712 0.059341372376 0.052720955999 rpy=-0.004379740805 -0.011997849886 0.001732382692
- joint r_elbow_flex_joint: limit lower=-2.1213 upper=-0.15 effort=30 velocity=3.3 -> lower=-2.3213 upper=0 effort=30 velocity=3.3
- joint r_forearm_cam_frame_joint: origin xyz=0.138338823418 -0.00626146937 0.044938792621 rpy=1.549884508472 -0.52315633191 0.0073610857 -> xyz=0.139183277238 0.002252222696 0.038145610345 rpy=1.569726130099 -0.540236735887 -0.022749929421
- joint r_gripper_l_finger_tip_joint: mimic (none) -> joint=r_gripper_l_finger_joint multiplier=1 offset=0
- joint r_gripper_r_finger_joint: mimic (none) -> joint=r_gripper_l_finger_joint multiplier=1 offset=0
- joint r_gripper_r_finger_tip_joint: mimic (none) -> joint=r_gripper_l_finger_joint multiplier=1 offset=0
- joint wide_stereo_frame_joint: origin xyz=0.039047869538 0.028900431683 0.045740529525 rpy=-0.006821150857 -0.011235489405 0.027024041802 -> xyz=0.04654507629 0.028051589334 0.052332857617 rpy=-0.005116533592 -0.016123200172 0.023786539594
